File: hardware/Volta-V1.kicad_sch (KiCad schematic)
At the start: 87 parts, among them SW1 TS-1088-AR02016, SW2 TS-1088-AR02016, U1 AMS1117-3.3, U2 CH32V317WCU6_C49188393, U3 SGL0622Z, U4 RDA5815M, X1 X50328MSB2GI, X2 Q13FC1350000400, X3 X49SD27MSD2SC

Commit message: AGC pin is now wired.
also have added a programming header section in the GPIO header.
Parts:
- added C28, C30: 0402B102K500NT, lcsc:C0402, symbol lcsc:0402B102K500NT
- added C36: CL05B104KO5NNNC, lcsc:C0402, symbol lcsc:CL05B104KO5NNNC
- added R14, R15, R9: 0402WGF2001TCE, lcsc:R0402, symbol lcsc:0402WGF2001TCE
- TP5: renamed from TP21; footprint TestPoint:TestPoint_Pad_D1.0mm -> lcsc:2xTinyTestPoint
- TP6: renamed from TP20; footprint TestPoint:TestPoint_Pad_D1.0mm -> lcsc:2xTinyTestPoint
- renumbered C8 to C1, C21 to C10, C15 to C12, C1 to C15, C3 to C16, C4 to C17, C2 to C18, C31 to C19, C16 to C2, C22 to C20, C23 to C21, C24 to C22, C32 to C23, C28 to C24, C27 to C25, C25 to C27, C33 to C29, C9 to C3, C30 to C31, C12 to C32, C5 to C33, C6 to C34, C7 to C35, C17 to C4, C18 to C5, C29 to C6, C19 to C7, C10 to C8, C20 to C9, L3 to L1, L4 to L2, L1 to L3, L2 to L4, R7 to R1, R9 to R12, R8 to R13, R12 to R2, R5 to R4, R4 to R5, R1 to R7, R2 to R8, SW2 to SW1, SW1 to SW2, TP9 to TP10, TP14 to TP11, TP18 to TP12, TP8 to TP14, TP17 to TP15, TP7 to TP16, TP16 to TP17, TP5 to TP18, TP4 to TP19, TP11 to TP2, TP3 to TP20, TP6 to TP21, TP2 to TP3, TP12 to TP4, TP10 to TP7, TP15 to TP8, TP19 to TP9, U4 to U2, U2 to U3, U3 to U4
Connections:
- net +3.3V: now also R15.2
- net GND: now also C28.1, C30.1
- net RF_FEED: now also C36.2; no longer L4.1, U4.1 (RF_OUT)
- net at U2.5 (AGC): now also C28.2, R9.2
- net GPIO_PE0 renamed RF_AGC
- net RF_AGC: now also R14.1, R15.1
- new net: C36.1, L4.1, U4.1 (RF_OUT)
- new net: C30.2, R14.2, R9.1
Other:
- note added: "TODO: * Check indication LED's GPIO pin"
- note removed: "TODO: * Wire AGC to PE0 (and add RC fitlers for PWM) * Check indication LED's GPIO pin"
- moved on the sheet: C20, C21, C22, C24, C25, C26, C27, JP1, R10, R11, R12, R13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

Commit message: finalize v1 and upload related documents
Changed lines of the file:
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@@
 	)
 	(junction
-		(at 414.02 110.49)
+		(at 411.48 110.49)
 		(diameter 0)
 		(color 0 0 0 0)
@@
 	(wire
 		(pts
-			(xy 415.29 147.32) (xy 415.29 151.13)
+			(xy 410.21 147.32) (xy 410.21 151.13)
 		)
 		(stroke
@@
 	(wire
 		(pts
-			(xy 379.73 110.49) (xy 414.02 110.49)
+			(xy 379.73 110.49) (xy 411.48 110.49)
 		)
 		(stroke
@@
 	(wire
 		(pts
-			(xy 414.02 110.49) (xy 414.02 113.03)
+			(xy 411.48 110.49) (xy 411.48 113.03)
 		)
 		(stroke
@@
 	(wire
 		(pts
-			(xy 414.02 106.68) (xy 414.02 110.49)
+			(xy 411.48 106.68) (xy 411.48 110.49)
 		)
 		(stroke
@@
 	(wire
 		(pts
-			(xy 394.97 151.13) (xy 415.29 151.13)
+			(xy 394.97 151.13) (xy 410.21 151.13)
 		)
 		(stroke
@@
 	(wire
 		(pts
-			(xy 379.73 113.03) (xy 414.02 113.03)
+			(xy 379.73 113.03) (xy 411.48 113.03)
 		)
 		(stroke
@@
 		(dnp no)
 		(property "Reference" "TP19"
-			(at 423.164 62.23 0)
+			(at 423.418 61.976 0)
 			(effects
 				(font
@@
 		)
 		(property "Value" "SDA"
-			(at 425.704 64.262 0)
+			(at 425.958 64.008 0)
 			(effects
 				(font
@@
 	(symbol
 		(lib_id "power:+3.3V")
-		(at 415.29 147.32 0)
+		(at 410.21 147.32 0)
 		(unit 1)
 		(exclude_from_sim no)
@@
 		(fields_autoplaced yes)
 		(property "Reference" "#PWR054"
-			(at 415.29 151.13 0)
+			(at 410.21 151.13 0)
 			(effects
 				(font
@@
 		)
 		(property "Value" "+3.3V"
-			(at 415.29 142.24 0)
+			(at 410.21 142.24 0)
 			(effects
 				(font
@@
 		)
 		(property "Footprint" ""
-			(at 415.29 147.32 0)
+			(at 410.21 147.32 0)
 			(effects
 				(font
@@
 		)
 		(property "Datasheet" ""
-			(at 415.29 147.32 0)
+			(at 410.21 147.32 0)
 			(effects
 				(font
@@
 		)
 		(property "Description" "Power symbol creates a global label with name \"+3.3V\""
-			(at 415.29 147.32 0)
+			(at 410.21 147.32 0)
 			(effects
 				(font
@@
 		(dnp no)
 		(property "Reference" "TP21"
-			(at 470.916 260.096 0)
+			(at 469.392 259.842 0)
 			(effects
 				(font
@@
 		)
 		(property "Value" "BIAS-T"
-			(at 474.726 262.128 0)
+			(at 473.964 261.874 0)
 			(effects
 				(font
@@
 		(dnp no)
 		(property "Reference" "TP20"
-			(at 428.244 59.69 0)
+			(at 429.26 57.912 0)
 			(effects
 				(font
@@
 		)
 		(property "Value" "AGC"
-			(at 430.784 61.722 0)
+			(at 431.8 59.944 0)
 			(effects
 				(font
@@
 	(symbol
 		(lib_id "power:+3.3V")
-		(at 414.02 106.68 0)
+		(at 411.48 106.68 0)
 		(unit 1)
 		(exclude_from_sim no)
@@
 		(fields_autoplaced yes)
 		(property "Reference" "#PWR052"
-			(at 414.02 110.49 0)
+			(at 411.48 110.49 0)
 			(effects
 				(font
@@
 		)
 		(property "Value" "+3.3V"
-			(at 414.02 101.6 0)
+			(at 411.48 101.6 0)
 			(effects
 				(font
@@
 		)
 		(property "Footprint" ""
-			(at 414.02 106.68 0)
+			(at 411.48 106.68 0)
 			(effects
 				(font
@@
 		)
 		(property "Datasheet" ""
-			(at 414.02 106.68 0)
+			(at 411.48 106.68 0)
 			(effects
 				(font
@@
 		)
 		(property "Description" "Power symbol creates a global label with name \"+3.3V\""
-			(at 414.02 106.68 0)
+			(at 411.48 106.68 0)
 			(effects
 				(font
